File: Eurorack_mini_psu.brd (EAGLE design)
At the start: 76.5 x 46.3 mm, 24 parts, among them IC1 7805TV

Commit message: Updates PCB labels.
Parts:
- moved R2 1.80 mm to (59.7, 43.2), turned to 0 degrees
- moved R3 1.80 mm to (47.0, 43.2), turned to 0 degrees
- turned LED1 to 90 degrees
- turned LED2 to 90 degrees
- turned LED3 to 90 degrees
- turned LED4 to 90 degrees
Routing:
- net +12V: track 100.1 -> 97.5 mm
- net N$10: track 7.40 -> 4.86 mm
- net N$11: track 8.67 -> 6.88 mm
- net N$13: track 3.81 -> 5.61 mm
- net -12V: track 107.2 -> 106.0 mm
- net +5V: track 87.8 -> 88.6 mm
- net N$7: track 3.81 -> 3.07 mm
Other:
- board text added: "EURORACK mini switching PSU"
- board text removed: "EURORACK mini PSU"
